Commit message: Fixed pendulum xacro include and fixed inertia problem

File: Simple-Pendulum/basic_sphere.xacro (robot description, xacro)
@@ -4,12 +4,13 @@
         <pose>${pos} ${rot}</pose>
         <inertial>
-        <mass>${mass}</mass>
-        <inertia>
-            <ixx>${2 * mass * (radius * radius)/3}</ixx>
-            <iyy>${2 * mass * (radius * radius)/3}</iyy>
-            <izz>${2 * mass * (radius * radius)/3}</izz>
-            <ixy>0</ixy>
-            <ixz>0</ixz>
-            <iyz>0</iyz>
+            <mass>${mass}</mass>
+            <inertia>
+                <ixx>${2 * mass * (radius * radius)/3}</ixx>
+                <iyy>${2 * mass * (radius * radius)/3}</iyy>
+                <izz>${2 * mass * (radius * radius)/3}</izz>
+                <ixy>0</ixy>
+                <ixz>0</ixz>
+                <iyz>0</iyz>
+            </inertia>
         </inertial>
         <visual name="visual">

File: Simple-Pendulum/world.xacro (robot description, xacro)
@@ -2,5 +2,5 @@
 <sdf version="1.7">
     <robot xmlns:xacro="http://www.ros.org/wiki/xacro">
-        <xacro:include filename="simple_pendulum_model.xacro" />
+        <xacro:include filename="pendulum.xacro" />
         <world name='default'>
             <include>
