Commit message: Made the pendulum not fall anymore

File: Simple-Pendulum/pendulum.xacro (robot description, xacro)
@@ -1,4 +1,5 @@
 <?xml version="1.0"?>
 <sdf version="1.7" xmlns:xacro="http://www.ros.org/wiki/xacro">
+    <xacro:property name="PI" value="3.14159" />
     <xacro:property name="arm_length" value="1.0" />
     <xacro:property name="bob_radius" value="0.05" />
@@ -7,22 +8,36 @@
     <xacro:property name="arm_mass" value="0.1" />
     <xacro:property name="bob_mass" value="0.5" />
-    <xacro:property name="base_radius" value="0.5" />
+    <xacro:property name="base_size_x" value="0.5" />
+    <xacro:property name="base_size_y" value="0.5" />
+    <xacro:property name="arm_holder_size_x" value="0.02" />
+    <xacro:property name="arm_holder_size_y" value="0.01" />
+    <xacro:property name="arm_holder_size_z" value="0.01" />
     <xacro:include filename="basic_sphere.xacro"/>
+    <xacro:include filename="basic_box.xacro"/>
     <xacro:include filename="basic_cylinder.xacro"/>
-    <xacro:macro name="simple_pendulum" params="x y z roll pitch yaw">
+    <xacro:macro name="simple_pendulum" params="x y z theta_0">
         <model name="simple_pendulum">
-            <pose>${x} ${y} ${z} ${roll} ${pitch} ${yaw}</pose>
-            <link name="base_link"/>
+            <pose>${x} ${y} ${z + 0.01} 0 0 0</pose>
+            <link name="base_link">
+                <xacro:basic_box pos="0 0 ${-z/2}" rot="0 0 0" mass="1000"
+                size_x="${base_size_x}" size_y="${base_size_y}" size_z="${z}"
+                color="0 0 1 1"/>
+            </link>
+            <link name="arm_holder">
+                <xacro:basic_box pos="${base_size_x} 0 0" rot="0 0 0" mass="0.1"
+                size_x="${arm_holder_size_x}" size_y="${arm_holder_size_y}"
+                size_z="${arm_holder_size_z}" color="0.5 0 0.5 1"/>
+            </link>
             <link name="arm">
-                <xacro:basic_cylinder pos="0 0 ${arm_length/2}"
+                <xacro:basic_cylinder pos="${arm_holder_size_x + base_size_x} 0 ${-arm_length/2}"
                     rot="0 0 0" mass="0.1" radius="${arm_radius}"
                     length="${arm_length}" color="1 0 0 1"/>
             </link>
             <link name="bob">
-                <xacro:basic_solid_sphere pos="0 0 ${arm_length}" rot="0 0 0"
+                <xacro:basic_solid_sphere pos="${arm_holder_size_x + base_size_x} 0 ${arm_length}" rot="0 0 0"
                 radius="${bob_radius}" color="0 1 0 1" mass="10"/>
             </link>
             <joint name="arm_joint" type="revolute">
-                <parent>base_link</parent>
+                <parent>arm_holder</parent>
                 <child>arm</child>
                 <axis>
@@ -35,4 +50,8 @@
                 <pose>0 0 0 0 0 0</pose>
             </joint>
+            <joint name="arm_holder_joint" type="fixed">
+                <parent>base_link</parent>
+                <child>arm_holder</child>
+            </joint>
             <joint name="bob_joint" type="fixed">
                 <parent>arm</parent>

File: Simple-Pendulum/world.xacro (robot description, xacro)
@@ -4,7 +4,7 @@
     <world name='default'>
         <include>
-            <uri> model://ground_plane </uri>
+            <uri>model://ground_plane</uri>
         </include>
-        <xacro:simple_pendulum x="0" y="0" z="2" roll="0" pitch="0" yaw="1.64"/>
+        <xacro:simple_pendulum x="0" y="0" z="2" roll="0" pitch="0" yaw="0"/>
     </world>
 </sdf>

Commit message: Fixed some compilation errors

File: Simple-Pendulum/pendulum.xacro (robot description, xacro)
@@ -2,5 +2,4 @@
 <sdf version="1.7" xmlns:xacro="http://www.ros.org/wiki/xacro">
     <xacro:property name="PI" value="3.14159" />
-    <xacro:property name="arm_length" value="1.0" />
     <xacro:property name="bob_radius" value="0.05" />
     <xacro:property name="base_radius" value="0.05" />
@@ -16,5 +15,5 @@
     <xacro:include filename="basic_box.xacro"/>
     <xacro:include filename="basic_cylinder.xacro"/>
-    <xacro:macro name="simple_pendulum" params="x y z theta_0">
+    <xacro:macro name="simple_pendulum" params="x y z theta_0 arm_length">
         <model name="simple_pendulum">
             <pose>${x} ${y} ${z + 0.01} 0 0 0</pose>
@@ -31,5 +30,5 @@
             <link name="arm">
                 <xacro:basic_cylinder pos="${arm_holder_size_x + base_size_x} 0 ${-arm_length/2}"
-                    rot="0 0 0" mass="0.1" radius="${arm_radius}"
+                    rot="${theta_0} 0 0" mass="0.1" radius="${arm_radius}"
                     length="${arm_length}" color="1 0 0 1"/>
             </link>

File: Simple-Pendulum/world.xacro (robot description, xacro)
@@ -6,5 +6,5 @@
             <uri>model://ground_plane</uri>
         </include>
-        <xacro:simple_pendulum x="0" y="0" z="2" roll="0" pitch="0" yaw="0"/>
+        <xacro:simple_pendulum x="0" y="0" z="2" theta_0="1.2" arm_length="1.0"/>
     </world>
 </sdf>

Commit message: Fixed ground plane problem

File: Simple-Pendulum/pendulum.xacro (robot description, xacro)
@@ -19,4 +19,5 @@
             <pose>${x} ${y} ${z + 0.01} 0 0 0</pose>
             <link name="base_link">
+                <static>true</static>
                 <xacro:basic_box pos="0 0 ${-z/2}" rot="0 0 0" mass="1000"
                 size_x="${base_size_x}" size_y="${base_size_y}" size_z="${z}"

File: Simple-Pendulum/world.xacro (robot description, xacro)
@@ -3,7 +3,29 @@
     <xacro:include filename="pendulum.xacro" />
     <world name='default'>
-        <include>
-            <uri>model://ground_plane</uri>
-        </include>
+        <model name="ground_plane">
+            <static>true</static>
+            <link name="link">
+                <collision name="collision">
+                <geometry>
+                    <plane>
+                    <normal>0 0 1</normal>
+                    </plane>
+                </geometry>
+                </collision>
+                <visual name="visual">
+                <geometry>
+                    <plane>
+                    <normal>0 0 1</normal>
+                    <size>100 100</size>
+                    </plane>
+                </geometry>
+                <material>
+                    <ambient>0.8 0.8 0.8 1</ambient>
+                    <diffuse>0.8 0.8 0.8 1</diffuse>
+                    <specular>0.8 0.8 0.8 1</specular>
+                </material>
+                </visual>
+            </link>
+        </model>
         <xacro:simple_pendulum x="0" y="0" z="2" theta_0="1.2" arm_length="1.0"/>
     </world>

Commit message: Fixed SDF fully

File: Simple-Pendulum/pendulum.xacro (robot description, xacro)
@@ -2,7 +2,7 @@
 <sdf version="1.7" xmlns:xacro="http://www.ros.org/wiki/xacro">
     <xacro:property name="PI" value="3.14159" />
-    <xacro:property name="bob_radius" value="0.05" />
+    <xacro:property name="bob_radius" value="0.1" />
     <xacro:property name="base_radius" value="0.05" />
-    <xacro:property name="arm_radius" value="0.01" />
+    <xacro:property name="arm_radius" value="0.03" />
     <xacro:property name="arm_mass" value="0.1" />
     <xacro:property name="bob_mass" value="0.5" />
@@ -24,15 +24,15 @@
             </link>
             <link name="arm_holder">
-                <xacro:basic_box pos="${(base_size_x+arm_holder_size_x)/2} 0 0" rot="${PI/2} 0 0" mass="0.1"
-                size_x="${(arm_holder_size_x + base_size_x)}" size_y="${arm_holder_size_y}"
-                size_z="${arm_holder_size_z}" color="0.5 0 0.5 1"/>
+                <xacro:basic_box pos="${(base_size_x+arm_holder_size_x)/4} 0 0" rot="0 0 0" mass="0.1"
+                size_x="${(arm_holder_size_x + base_size_x)/2}" size_y="${arm_holder_size_y}"
+                size_z="${arm_holder_size_z}" color="0 0 1 1"/>
             </link>
             <link name="arm">
-                <xacro:basic_cylinder pos="${arm_holder_size_x + base_size_x} 0 ${-arm_length/2}"
-                    rot="0 0 0" mass="0.1" radius="${arm_radius}"
+                <xacro:basic_cylinder pos="${arm_holder_size_x + base_size_x/2} ${arm_length/2} 0"
+                    rot="${PI/2} 0 0" mass="0.1" radius="${arm_radius}"
                     length="${arm_length}" color="1 0 0 1"/>
             </link>
             <link name="bob">
-                <xacro:basic_solid_sphere pos="0 ${arm_holder_size_x + base_size_x} 0" rot="0 0 0"
+                <xacro:basic_solid_sphere pos="${arm_holder_size_x + base_size_x/2} ${arm_length} 0" rot="0 0 0"
                 radius="${bob_radius}" color="0 1 0 1" mass="10"/>
             </link>
@@ -40,7 +40,7 @@
                 <parent>arm_holder</parent>
                 <child>arm</child>
+                <pose>0 0 ${arm_length/2} 0 0 0</pose>
                 <axis>
-                    <xyz>0 1 0</xyz>
-                    <pose>0 0 0 0 0 0</pose>
+                    <xyz>1 0 0</xyz>
                     <limit>
                         <lower>-1e16</lower>

File: Simple-Pendulum/world.xacro (robot description, xacro)
@@ -2,31 +2,8 @@
 <sdf version="1.7" xmlns:xacro="http://www.ros.org/wiki/xacro">
     <xacro:include filename="pendulum.xacro" />
+    <xacro:include filename="ground_plane.xacro" />
     <world name='default'>
-        <model name="ground_plane">
-            <static>true</static>
-            <link name="link">
-                <collision name="collision">
-                <geometry>
-                    <plane>
-                    <normal>0 0 1</normal>
-                    </plane>
-                </geometry>
-                </collision>
-                <visual name="visual">
-                <geometry>
-                    <plane>
-                    <normal>0 0 1</normal>
-                    <size>100 100</size>
-                    </plane>
-                </geometry>
-                <material>
-                    <ambient>0.8 0.8 0.8 1</ambient>
-                    <diffuse>0.8 0.8 0.8 1</diffuse>
-                    <specular>0.8 0.8 0.8 1</specular>
-                </material>
-                </visual>
-            </link>
-        </model>
-        <xacro:simple_pendulum x="0" y="0" z="2" theta_0="1.2" arm_length="1.0"/>
+        <xacro:ground_plane/>
+        <xacro:simple_pendulum x="0" y="0" z="1.3" theta_0="1.2" arm_length="1.0"/>
     </world>
 </sdf>
